File: hardware/Quadrotor/Quadrotor.sch (KiCad schematic (older format))
At the start: 118 parts, among them J1 Power, J10 MotorD, J2 EX_EXM, J3 EX_SPI, J4 USB_B_Micro, J5 MCU_JTAG, J6 NRF_JA, J7 MotorA, J8 MotorC, J9 MotorB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

Commit message: PCB布板完成
Parts:
- removed TP5: MPU_SDA, TestPoint:TestPoint_Pad_D1.0mm, symbol Connector:TestPoint
- removed TP6: MPU_SCL, TestPoint:TestPoint_Pad_D1.0mm, symbol Connector:TestPoint
Connections:
- wire segments 267 -> 264
Other:
- moved on the sheet: R3, SW1
Changed lines of the file:
@@
 EESchema Schematic File Version 4
+LIBS:Quadrotor-cache
 EELAYER 29 0
 EELAYER END
@@
 	-1   0    0    1
 $EndComp
-Wire Wire Line
-	7100 4575 7350 4575
 $Comp
 L Quadrotor:+3V #PWR0136
@@
 L Switch:SW_Push SW1
 U 1 1 5F007DD7
-P 15175 2800
-F 0 "SW1" H 15175 3000 50  0000 C CNN
-F 1 "SW_Push" H 15350 2925 50  0000 C CNN
-F 2 "Button_Switch_SMD:SW_SPST_PTS810" H 15175 3000 50  0001 C CNN
-F 3 "~" H 15175 3000 50  0001 C CNN
-	1    15175 2800
+P 15175 5800
+F 0 "SW1" H 15175 6000 50  0000 C CNN
+F 1 "SW_Push" H 15350 5925 50  0000 C CNN
+F 2 "Button_Switch_SMD:SW_SPST_PTS810" H 15175 6000 50  0001 C CNN
+F 3 "~" H 15175 6000 50  0001 C CNN
+	1    15175 5800
 	1    0    0    -1
 $EndComp
@@
 L Device:R_Small R3
 U 1 1 5F00890C
-P 14925 2525
-F 0 "R3" H 15025 2575 50  0000 C CNN
-F 1 "10K" H 15025 2500 50  0000 C CNN
-F 2 "Resistor_SMD:R_0402_1005Metric" H 14925 2525 50  0001 C CNN
-F 3 "~" H 14925 2525 50  0001 C CNN
-	1    14925 2525
-	1    0    0    -1
-$EndComp
-Wire Wire Line
-	14975 2800 14925 2800
-Wire Wire Line
-	14925 2800 14925 2625
-Wire Wire Line
-	14925 2425 14925 1850
-Wire Wire Line
-	14925 2800 14525 2800
-Connection ~ 14925 2800
+P 14925 5525
+F 0 "R3" H 15025 5575 50  0000 C CNN
+F 1 "10K" H 15025 5500 50  0000 C CNN
+F 2 "Resistor_SMD:R_0402_1005Metric" H 14925 5525 50  0001 C CNN
+F 3 "~" H 14925 5525 50  0001 C CNN
+	1    14925 5525
+	1    0    0    -1
+$EndComp
+Wire Wire Line
+	14975 5800 14925 5800
+Wire Wire Line
+	14925 5800 14925 5625
+Wire Wire Line
+	14925 5800 14525 5800
+Connection ~ 14925 5800
 $Comp
 L power:GNDD #PWR0162
 U 1 1 5F048A32
-P 15375 2800
-F 0 "#PWR0162" H 15375 2550 50  0001 C CNN
-F 1 "GNDD" V 15379 2690 50  0000 R CNN
-F 2 "" H 15375 2800 50  0001 C CNN
-F 3 "" H 15375 2800 50  0001 C CNN
-	1    15375 2800
+P 15375 5800
+F 0 "#PWR0162" H 15375 5550 50  0001 C CNN
+F 1 "GNDD" V 15379 5690 50  0000 R CNN
+F 2 "" H 15375 5800 50  0001 C CNN
+F 3 "" H 15375 5800 50  0001 C CNN
+	1    15375 5800
 	0    -1   -1   0
 $EndComp
@@
 	11850 3375 12200 3375
 Connection ~ 12200 3375
-Wire Wire Line
-	12200 3075 12550 3075
-Wire Wire Line
-	12550 3075 12550 3300
-Wire Wire Line
-	12550 3300 12725 3300
-Connection ~ 12200 3075
-Wire Wire Line
-	12725 3100 12725 2775
-Wire Wire Line
-	12725 2775 12200 2775
 $Comp
 L power:GNDD #PWR0165
@@
 	0    1    1    0
 $EndComp
-Wire Wire Line
-	6600 4775 6850 4775
 $Comp
 L Quadrotor:+3V #PWR0137
@@
 	1    0    0    -1
 $EndComp
-$Comp
-L Connector:TestPoint TP5
-U 1 1 5FE6CD8B
-P 7350 4575
-F 0 "TP5" H 7408 4693 50  0000 L CNN
-F 1 "MPU_SDA" H 7400 4625 50  0000 L CNN
-F 2 "TestPoint:TestPoint_Pad_D1.0mm" H 7550 4575 50  0001 C CNN
-F 3 "~" H 7550 4575 50  0001 C CNN
-	1    7350 4575
-	1    0    0    -1
-$EndComp
-Connection ~ 7350 4575
-Wire Wire Line
-	7350 4575 7950 4575
-$Comp
-L Connector:TestPoint TP6
-U 1 1 5FEC3195
-P 6850 4775
-F 0 "TP6" H 6908 4893 50  0000 L CNN
-F 1 "MPU_SCL" H 6900 4825 50  0000 L CNN
-F 2 "TestPoint:TestPoint_Pad_D1.0mm" H 7050 4775 50  0001 C CNN
-F 3 "~" H 7050 4775 50  0001 C CNN
-	1    6850 4775
-	1    0    0    -1
-$EndComp
-Connection ~ 6850 4775
-Wire Wire Line
-	6850 4775 7950 4775
 $Comp
 L Quadrotor:+3V #PWR0149
@@
 	1    0    0    -1
 $EndComp
-Connection ~ 14425 1850
-Wire Wire Line
-	14425 1850 14925 1850
 Wire Wire Line
 	13925 1850 14425 1850
@@
 NoConn ~ 14525 5600
 NoConn ~ 14525 5700
-NoConn ~ 14525 5800
+NoConn ~ 14525 2800
 NoConn ~ 14525 5900
 $Comp
@@
 Wire Wire Line
 	12200 2775 12100 2775
-Connection ~ 12200 2775
 NoConn ~ 3375 4375
 NoConn ~ 3375 4475
@@
 	1    0    0    -1
 $EndComp
+$Comp
+L Quadrotor:+3V #PWR?
+U 1 1 5E506CD4
+P 14925 5425
+F 0 "#PWR?" H 14925 5275 50  0001 C CNN
+F 1 "+3V" H 14940 5598 50  0000 C CNN
+F 2 "" H 14925 5425 50  0001 C CNN
+F 3 "" H 14925 5425 50  0001 C CNN
+	1    14925 5425
+	1    0    0    -1
+$EndComp
+Wire Wire Line
+	6600 4775 7950 4775
+Wire Wire Line
+	7100 4575 7950 4575
+Wire Wire Line
+	12725 3100 12550 3100
+Wire Wire Line
+	12550 3100 12550 3075
+Wire Wire Line
+	12550 3075 12200 3075
+Connection ~ 12200 3075
+Wire Wire Line
+	12475 3300 12475 2775
+Wire Wire Line
+	12475 2775 12200 2775
+Wire Wire Line
+	12475 3300 12725 3300
+Connection ~ 12200 2775
 $EndSCHEMATC
